File: Demo_Board_Kicad/Demo_Board_Kicad.kicad_pcb (KiCad board)
At the start: 2 copper layers, 100 x 50 mm, 48 parts, among them J1 Power_IN, J2 POWER_OUT, J3 i2c Connector, J4 DBG_enable, J5 DBG_Voltage, J6 DBG_Sense, J7 Power, J8 Button Connector, J9 DIP_Address, Q1 Q_NMOS_DGS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

Commit message: reworked pcb and added new files
Parts:
- removed J4: DBG_enable, Pin_Headers:Pin_Header_Straight_1x02_Pitch2.54mm
- removed J5: DBG_Voltage, Pin_Headers:Pin_Header_Straight_1x02_Pitch2.54mm
- removed J6: DBG_Sense, Pin_Headers:Pin_Header_Straight_1x02_Pitch2.54mm
- added C10: 10uF, Capacitors_SMD:C_0603_HandSoldering, F.Cu at (225.3, 102.8)
- added C7: 100nF, Capacitors_SMD:C_0603_HandSoldering, F.Cu at (227.0, 90.6)
- added C8: 100nF, Capacitors_SMD:C_0603_HandSoldering, F.Cu at (220.0, 93.4)
- added C9: 22uF, Capacitors_SMD:C_0603_HandSoldering, F.Cu at (225.3, 98.8)
- added J10: i2c Internal, Pin_Headers:Pin_Header_Straight_1x02_Pitch2.54mm, F.Cu at (210.4, 88.6)
- added R20: 10k, Resistors_SMD:R_0603_HandSoldering, F.Cu at (216.7, 91.4)
- added R21: 10k, Resistors_SMD:R_0603_HandSoldering, F.Cu at (214.7, 90.1)
- added U5: ISO1540D, Housings_SOIC:SOIC-8_3.9x4.9mm_Pitch1.27mm, F.Cu at (221.7, 89.7)
- added U6: AZ1117CH-5.0TRG1, TO_SOT_Packages_SMD:SOT-223-3Lead_TabPin2, F.Cu at (231.3, 101.5)
- C1: value 100uF -> 10uF; footprint Capacitors_THT:CP_Radial_D6.3mm_P2.50mm -> Capacitors_SMD:C_0603_HandSoldering
- J3: value i2c Connector -> i2c_iso_conn; footprint Pin_Headers:Pin_Header_Straight_1x06_Pitch2.54mm -> Pin_Headers:Pin_Header_Straight_1x04_Pitch2.54mm
- moved R14 43.8 mm to (195.1, 104.1)
- moved R15 42.5 mm to (195.1, 102.2)
- moved J9 42.2 mm to (201.8, 91.5), turned to 90 degrees
- moved R5 31.4 mm to (211.1, 105.7)
- moved R4 28.8 mm to (212.2, 109.0), turned to 0 degrees
- moved C5 27.0 mm to (207.6, 103.6)
- moved J3 26.7 mm to (232.2, 88.8)
- moved U1 26.3 mm to (202.3, 105.2)
- moved R16 15.1 mm to (178.6, 90.7), turned to 90 degrees
- moved R6 15.1 mm to (239.8, 98.3)
- moved R12 13.7 mm to (191.3, 98.4), turned to 180 degrees
- moved C4 13.0 mm to (180.8, 90.4), turned to 270 degrees
- moved R2 13.0 mm to (201.9, 113.9)
- moved D3 12.9 mm to (244.8, 98.3), turned to 180 degrees
- moved J7 11.4 mm to (241.2, 101.5), turned to 270 degrees
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Connections:
- C1 pad 1: +5V -> +5VA
- C1 pad 2: GND -> GNDA
- J3 pad 1: GND -> GNDA
- J3 pad 2: GND -> /SCL_iso
- J3 pad 3: /SCL -> /SDA_iso
- J3 pad 4: /SDA -> +5VA
- J8 pad 2: /BTN_Clock -> /LED_Purple
- J8 pad 3: /LED_Purple -> /LED_Red
- J8 pad 4: /LED_Red -> /LED_Green
- J8 pad 5: /LED_Green -> /BTN_Clock
- U1 pad 13: /TempSense -> /OutVoltage
- U1 pad 3: /OutVoltage -> /TempSense
- U2 pad 1: /Adr0_SEL -> /Adr1_SEL
- U2 pad 10: /LED_Green -> /LED_Red
- U2 pad 11: /LED_Red -> /LED_Purple
- U2 pad 12: /LED_Purple -> /LED_DEBUG
- U2 pad 2: /Adr1_SEL -> /Adr0_SEL
- U2 pad 5: /BTN_Latch -> /BTN_Clock
- U2 pad 6: /BTN_Clock -> /BTN_Reset
- U2 pad 7: /BTN_Reset -> /BTN_Latch
- U2 pad 9: /LED_DEBUG -> /LED_Green
Routing:
- net +5V: track 198.2 -> 130.2 mm, vias 10 -> 8
- net /Adr0_SEL: track 70.4 -> 23.9 mm, vias 7 -> 4
- net /OutVoltage: track 58.2 -> 12.6 mm, vias 5 -> 0
- net /Adr1_SEL: track 60.5 -> 25.8 mm, vias 7 -> 4
- net GND: track 43.5 -> 9.88 mm, vias 1 -> 0
- net +5VA: track 0.00 -> 16.6 mm
- net /SDA_iso: track 0.00 -> 13.8 mm
- net /LED_Purple: track 31.1 -> 17.7 mm
- net /BTN_Latch: track 22.9 -> 10.1 mm, vias 4 -> 2
- net /BTN_Clock: track 42.8 -> 30.6 mm, vias 2 -> 4
- net /SCL_iso: track 0.00 -> 11.5 mm, vias 0 -> 1
- net /LED_Red: track 27.0 -> 16.5 mm
- net /OutEnable: track 42.6 -> 32.7 mm, vias 3 -> 4
- net /LED_Green: track 23.2 -> 13.6 mm
- net GNDA: track 0.00 -> 9.54 mm
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