File: Demo_Board_Kicad/Demo_Board_Kicad.sch (KiCad schematic (older format))
At the start: 48 parts, among them J1 Power_IN, J2 POWER_OUT, J3 i2c Connector, J4 DBG_enable, J5 DBG_Voltage, J6 DBG_Sense, J7 Power, J8 Button Connector, J9 DIP_Address, Q1 Q_NMOS_DGS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

Commit message: reworked pcb and added new files
Parts:
- removed C1: 100uF, Capacitors_THT:CP_Radial_D6.3mm_P2.50mm, symbol CP
- removed J3: i2c Connector, Pin_Headers:Pin_Header_Straight_1x06_Pitch2.54mm, symbol CONN_01X06
- added C1, C10: 10uF, Capacitors_SMD:C_0603_HandSoldering, symbol C_Small
- added C7, C8: 100nF, Capacitors_SMD:C_0603_HandSoldering, symbol C_Small
- added C9: 22uF, Capacitors_SMD:C_0603_HandSoldering, symbol C_Small
- added J10: i2c Internal, Pin_Headers:Pin_Header_Straight_1x02_Pitch2.54mm, symbol CONN_01X02
- added J3: i2c_iso_conn, Pin_Headers:Pin_Header_Straight_1x04_Pitch2.54mm, symbol CONN_01X04
- added R20, R21: 10k, Resistors_SMD:R_0603_HandSoldering, symbol R_Small
- added U5: ISO1540D, Housings_SOIC:SOIC-8_3.9x4.9mm_Pitch1.27mm, symbol ISO1540D
- added U6: AZ1117CH-5.0TRG1, TO_SOT_Packages_SMD:SOT-223-3Lead_TabPin2, symbol AZ1117CH-5.0TRG1
Connections:
- net +5V: now also C8.2, C9.2, R20.1, R21.2, U5.8 (VCC2), U6.2 (OUTPUT)
- net +BATT: now also C10.2, U6.3 (INPUT)
- net Adr0_SEL: now also U2.2 (A1); no longer U2.1 (A0)
- net Adr1_SEL: now also U2.1 (A0); no longer U2.2 (A1)
- net BTN_Clock: now also J8.5 (P5), U2.5 (IO_1); no longer J8.2 (P2), U2.6 (IO_2)
- net BTN_Latch: now also U2.7 (IO_3); no longer U2.5 (IO_1)
- net BTN_Reset: now also U2.6 (IO_2); no longer U2.7 (IO_3)
- net GND: now also C10.1, C8.1, C9.1, U5.5 (GND2), U6.1 (GND)
- net LED_DEBUG: now also U2.12 (IO_7); no longer U2.9 (IO_4)
- net LED_Green: now also J8.4 (P4), U2.9 (IO_4); no longer J8.5 (P5), U2.10 (IO_5)
- net LED_Purple: now also J8.2 (P2), U2.11 (IO_6); no longer J8.3 (P3), U2.12 (IO_7)
- net LED_Red: now also J8.3 (P3), U2.10 (IO_5); no longer J8.4 (P4), U2.11 (IO_6)
- net OutVoltage: now also U1.13 (CH4+); no longer U1.3 (CH2+)
- net SCL: now also J10.1 (P1), R21.1, U5.6 (SCL2)
- net SDA: now also J10.2 (P2), R20.2, U5.7 (SDA2)
- net TempSense: now also U1.3 (CH2+); no longer U1.13 (CH4+)
- new net +5VA: C1.1, C7.2, J3.4 (P4), U5.1 (VCC1)
- new net GNDA: C1.2, C7.1, J3.1 (P1), U5.4 (GND1)
- new net SCL_iso: J3.2 (P2), U5.3 (SCL1)
- new net SDA_iso: J3.3 (P3), U5.2 (SDA1)
Other:
- note added: "5V Regulator\nmaybe choose one with higher input rating?"
- note added: "Powerfet"
- note added: "i2c Isolator"
- note added: "i2c Pull Up"
- moved on the sheet: D2, J9, Q1, Q3, R12, R14, R15, R2, R3
